File: CAO-electronic/LedsBoard/LedsBoard.kicad_sch (KiCad schematic)
At the start: 22 parts

Commit message: first proto
Parts:
- added FB1: 100Ω, Inductor_SMD:L_0603_1608Metric, symbol TrucPourPlantes:BLM18KN101EH1D
- added J1: ~, TrucPourPlantes:Würth_WR-WTB_620109131822_1x09_P2.00mm_Horizontal, symbol TrucPourPlantes:620109131822
- renumbered Q5 to Q2, Q2 to Q3, Q3 to Q4, Q4 to Q5, R3 to R1, R9 to R10, R10 to R11, R11 to R12, R12 to R13, R1 to R3, R13 to R4, R4 to R5, R5 to R6, R6 to R7, R7 to R8, R8 to R9
Connections:
- net +5V: now also FB1.1, J1.1 (Pin_1), J1.2 (Pin_2); no longer Q2.2 (C)
- net GND: now also J1.8 (Pin_8), J1.9 (Pin_9), J1.MP (MountPin)
- net Led_Deep_Blue: now also J1.5 (Pin_5)
- net Led_Far_Red: now also J1.4 (Pin_4)
- net Led_High_Red: now also J1.3 (Pin_3)
- net Led_White: now also J1.6 (Pin_6)
- net Light_Signal: now also J1.7 (Pin_7)
- new net: FB1.2, Q2.2 (C)
